File: CANBoard/CANBoard.kicad_pcb (KiCad board)
At the start: 4 copper layers, 40 x 40 mm, 83 parts, among them J1 Conn_01x08, J2 Conn_01x08, J3 Conn_01x08, J4 Conn_01x08, J5 TC2030, Q1 DMN2004WK, Q2 DMN2004WK, Q3 DMN2004WK, Q4 DMN2004WK, U1 TPS56339DDCR, U2 LD1117S33CTR, U3 MCP2562, U4 STM32F303K8T6, Y1 8mHz

Commit message: move footprints to project library
Parts:
- D2: footprint digikey-footprints:SOT-23-3 -> CANBoard:SOT-23-3
- G1: footprint DRTLogo:DRTLogo -> CANBoard:DRTLogo
- G2: footprint DRTLogo:DingoFaceNoFill -> CANBoard:DingoFaceNoFill
- U1: footprint TO_SOT_SMD_Modify:SOT-23-6_NoPin5 -> CANBoard:SOT-23-6_NoPin5
- U2: footprint digikey-footprints:SOT-223 -> CANBoard:SOT-223
