File: CANBoard/CANBoard.kicad_sch (KiCad schematic)
At the start: 25 parts, among them J1 Conn_01x08, J2 Conn_01x08, J3 Conn_01x08, J4 Conn_01x08, U1 TPS56339DDCR, U2 LD1117S33CTR

Commit message: move footprints to project library
Parts:
- G1: footprint DRTLogo:DRTLogo -> CANBoard:DRTLogo
- G2: footprint DRTLogo:DingoFaceNoFill -> CANBoard:DingoFaceNoFill
- U1: footprint TO_SOT_SMD_Modify:SOT-23-6_NoPin5 -> CANBoard:SOT-23-6_NoPin5
- U2: footprint digikey-footprints:SOT-223 -> CANBoard:SOT-223
Changed lines of the file:
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@@
 			)
 		)
-		(property "Footprint" "DRTLogo:DRTLogo"
+		(property "Footprint" "CANBoard:DRTLogo"
 			(at 265.43 135.89 0)
 			(effects
@@
 			)
 		)
-		(property "Footprint" "DRTLogo:DingoFaceNoFill"
+		(property "Footprint" "CANBoard:DingoFaceNoFill"
 			(at 265.43 142.24 0)
 			(effects
@@
 			)
 		)
-		(property "Footprint" "TO_SOT_SMD_Modify:SOT-23-6_NoPin5"
+		(property "Footprint" "CANBoard:SOT-23-6_NoPin5"
 			(at 129.54 30.48 0)
 			(effects
@@
 			)
 		)
-		(property "Footprint" "digikey-footprints:SOT-223"
+		(property "Footprint" "CANBoard:SOT-223"
 			(at 225.425 29.21 0)
 			(effects
