File: CANBoard/MCU.kicad_sch (KiCad schematic)
At the start: 23 parts, among them J5 TC2030, U3 MCP2562, U4 STM32F303K8T6, Y1 8mHz

Commit message: move footprints to project library
Parts:
- D2: footprint digikey-footprints:SOT-23-3 -> CANBoard:SOT-23-3
Changed lines of the file:
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@@
 			)
 		)
-		(property "Footprint" "digikey-footprints:SOT-23-3"
+		(property "Footprint" "CANBoard:SOT-23-3"
 			(at 144.145 182.245 0)
 			(effects
